Commit message: plant v2: vendor asimov-1 fix/ankle-roll 346e6cc; 23-hinge layout; qpos joint convention
- rgmt/assets/asimov-v1: MJCF/URDF byte-identical to upstream 346e6cc
  (neck welded, new foot mass/contact spheres, URDF torque caps 2.4-3.6x
  lower, elbow ref baked into the URDF origin), ANKLE_B_NEW.STL added,
  UPSTREAM note records the commit.
- NewtonSim: hinge columns are the REVOLUTE joints only (the welded neck
  imports as FIXED joints with no coordinates and would alias the next
  joint); n_hinges replaces every literal 25. The MJCF <option> block is
  not parsed; cone=pyramidal/impratio=1 are pinned in SolverMuJoCo so
  the contact model equals the released policy's.
- Joint angles above the sim are MuJoCo qpos everywhere: joint_q returns
  Newton angle + ref, reset_idx subtracts it, step() passes targets
  through. The retargeted clips are raw qpos (0 = straight elbow); the
  old ref compensation had bent every elbow 45 deg past the mocap.
- PASSIVE_JOINT_NAMES is empty; tests updated (URDF movable joints ==
  actuated set, new effort values, torque-starvation test compares envs
  at 2 s because the all-zeros pose topples backward on this asset).

Plant v1 (old asset, old caps, old convention) is tagged plant-v1.

Co-Authored-By: Claude Fable 5.1 <noreply@anthropic.com>
Claude-Session: https://claude.ai/code/session_01Jq5bQdUV6BGq9YmwWPyXtr

File: rgmt/assets/asimov-v1/xmls/asimov.urdf (robot description, URDF)
Before this commit: robot asimov, 26 links, 25 joints
Links:
- link left_ankle_pitch_link: mass 0.273090119400173 -> 0.2730901194
- link left_ankle_roll_link: mass 0.405640437504617 -> 0.44468; geometry collision sphere radius=0.005; collision sphere radius=0.005
- link left_elbow_link: mass 0.662317601299901 -> 0.6623176013; geometry collision cylinder length=0.1140175425 radius=0.03; collision sphere radius=0.03
- link left_hip_pitch_link: mass 1.05630112217695 -> 1.056301122; geometry collision cylinder length=0.02 radius=0.04; collision sphere radius=0.04
- link left_hip_roll_link: mass 0.414368139397033 -> 0.4143681394
- link left_hip_yaw_link: mass 1.86657016436158 -> 1.866570164; geometry collision cylinder length=0.07 radius=0.04; collision sphere radius=0.04
- link left_knee_link: mass 2.39114151033076 -> 2.391141511; geometry collision cylinder length=0.18 radius=0.04; collision sphere radius=0.04
- link left_shoulder_pitch_link: mass 0.599157136550892 -> 0.5991571366
- link left_shoulder_roll_link: mass 1.3132281302001 -> 1.31322813; geometry collision cylinder length=0.09 radius=0.035; collision sphere radius=0.035
- link left_shoulder_yaw_link: mass 0.712261755331765 -> 0.7122617553
- link left_wrist_yaw_link: mass 0.058058790654763 -> 0.05805879065; geometry visual mesh filename=../assets/meshes/LEFT_WRIST_YAW.STL
- link neck_pitch_link: mass 0.394055609177456 -> 0.3940556092; geometry collision cylinder length=0.04 radius=0.05; collision sphere radius=0.05
- link neck_yaw_link: mass 0.53278930532821 -> 0.5327893053
- link pelvis_link: mass 3.50691251175897 -> 3.506912512; geometry collision cylinder length=0.075 radius=0.04; collision sphere radius=0.04
- link right_ankle_pitch_link: mass 0.27308917159726 -> 0.2730891716
- link right_ankle_roll_link: mass 0.405640437504617 -> 0.44468; geometry collision sphere radius=0.005; collision sphere radius=0.005
- link right_elbow_link: mass 0.662314258886328 -> 0.6623142589; geometry collision cylinder length=0.1140175425 radius=0.03; collision sphere radius=0.03
- link right_hip_pitch_link: mass 1.05629742879001 -> 1.056297429; geometry collision cylinder length=0.02 radius=0.04; collision sphere radius=0.04
- link right_hip_roll_link: mass 0.414825000619808 -> 0.4148250006
- link right_hip_yaw_link: mass 1.86647220449567 -> 1.866472204; geometry collision cylinder length=0.07 radius=0.04; collision sphere radius=0.04
- link right_knee_link: mass 2.39110172735043 -> 2.391101676; geometry collision cylinder length=0.18 radius=0.04; collision sphere radius=0.04
- link right_shoulder_pitch_link: mass 0.599156105726411 -> 0.5991561057
- link right_shoulder_roll_link: mass 1.31322237625579 -> 1.313222376; geometry collision cylinder length=0.09 radius=0.035; collision sphere radius=0.035
- link right_shoulder_yaw_link: mass 0.712261755331765 -> 0.7122617553
- link right_wrist_yaw_link: mass 0.0580595106779709 -> 0.05805951068; geometry visual mesh filename=../assets/meshes/RIGHT_WRIST_YAW.STL
- link waist_yaw_link: mass 8.20850158063177 -> 8.208501581; geometry collision cylinder length=0.25 radius=0.06; collision sphere radius=0.06
Joints:
- removed joint neck_pitch_joint
- removed joint neck_yaw_joint
- added joint neck_pitch_link_fixed: type fixed, parent neck_yaw_link, child neck_pitch_link, origin xyz=0 0 0.03735 rpy=0 0 0
- added joint neck_yaw_link_fixed: type fixed, parent waist_yaw_link, child neck_yaw_link, origin xyz=-0.01659877455 0 0.3781670296 rpy=0 0 0
- joint left_ankle_pitch_joint: limit lower=-0.35 upper=0.35 effort=145 velocity=10 -> lower=-0.35 upper=0.35 effort=40 velocity=9.32; origin xyz=-0.00151572865907394 -0.000435034718868785 -0.272344184376349 rpy=0 0 0 -> xyz=-0.001515728659 -0.0004350347189 -0.2723441844 rpy=0 0 0
- joint left_ankle_roll_joint: limit lower=-0.35 upper=0.35 effort=57 velocity=10 -> lower=-0.35 upper=0.35 effort=17 velocity=9.32
- joint left_elbow_joint: limit lower=0 upper=2.443461 effort=36 velocity=10 -> lower=0 upper=2.443461 effort=12 velocity=9.32; origin xyz=0 0 -0.0963013 rpy=0 0 0 -> xyz=0 0 -0.0963013 rpy=0 0.785398 0
- joint left_hip_pitch_joint: limit lower=-2.094395 upper=1 effort=120 velocity=10 -> lower=-2.094395 upper=1 effort=45 velocity=12.57
- joint left_hip_roll_joint: limit lower=-0.785398 upper=0.785398 effort=90 velocity=10 -> lower=-0.785398 upper=0.785398 effort=45 velocity=3.98
- joint left_hip_yaw_joint: limit lower=-0.785398 upper=0.785398 effort=60 velocity=10 -> lower=-0.785398 upper=0.785398 effort=28 velocity=5.45; origin xyz=-0.04225 0.00700892571037183 -0.0515254787497069 rpy=0 0 0 -> xyz=-0.04225 0.00700892571 -0.05152547875 rpy=0 0 0
- joint left_knee_joint: limit lower=0 upper=1.5 effort=75 velocity=10 -> lower=0 upper=1.5 effort=45 velocity=12.25; origin xyz=0.00151572865906509 -0.00657389099150725 -0.218432672960972 rpy=0 0 0 -> xyz=0.001515728659 -0.006573890992 -0.218432673 rpy=0 0 0
- joint left_shoulder_pitch_joint: limit lower=-3.141593 upper=0.872665 effort=90 velocity=10 -> lower=-3.141593 upper=0.872665 effort=30 velocity=3.98
- joint left_shoulder_roll_joint: limit lower=-1.570796 upper=0 effort=75 velocity=10 -> lower=-1.570796 upper=0 effort=25 velocity=12.25
- joint left_shoulder_yaw_joint: limit lower=-1.570796 upper=1.570796 effort=60 velocity=10 -> lower=-1.570796 upper=1.570796 effort=20 velocity=5.45
- joint left_wrist_yaw_joint: limit lower=-3.141593 upper=3.141593 effort=36 velocity=10 -> lower=-3.141593 upper=3.141593 effort=12 velocity=9.32
- joint right_ankle_pitch_joint: limit lower=-0.35 upper=0.35 effort=145 velocity=10 -> lower=-0.35 upper=0.35 effort=40 velocity=9.32; origin xyz=-0.00151572865907394 0.000435034718868785 -0.272344184376349 rpy=0 0 0 -> xyz=-0.0015157 0.00053505 -0.27234 rpy=0 0 0
- joint right_ankle_roll_joint: limit lower=-0.35 upper=0.35 effort=57 velocity=10 -> lower=-0.35 upper=0.35 effort=17 velocity=9.32
- joint right_elbow_joint: limit lower=-2.443461 upper=0 effort=36 velocity=10 -> lower=-2.443461 upper=0 effort=12 velocity=9.32; origin xyz=0 0 -0.0966013 rpy=0 0 0 -> xyz=0 0 -0.0966013 rpy=0 0.785398 0
- joint right_hip_pitch_joint: limit lower=-1 upper=2.094395 effort=120 velocity=10 -> lower=-1 upper=2.094395 effort=45 velocity=12.57
- joint right_hip_roll_joint: limit lower=-0.785398 upper=0.785398 effort=90 velocity=10 -> lower=-0.785398 upper=0.785398 effort=45 velocity=3.98; origin xyz=0.0422501 -0.0400002759400924 0 rpy=0 0 0 -> xyz=0.04225 -0.04 0 rpy=0 0 0
- joint right_hip_yaw_joint: limit lower=-0.785398 upper=0.785398 effort=60 velocity=10 -> lower=-0.785398 upper=0.785398 effort=28 velocity=5.45; origin xyz=-0.04225 -0.00700892571037183 -0.0515254787497069 rpy=0 0 0 -> xyz=-0.04225 -0.0064271 -0.051601 rpy=0 0 0
- joint right_knee_joint: limit lower=-1.5 upper=0 effort=75 velocity=10 -> lower=-1.5 upper=0 effort=45 velocity=12.25; origin xyz=0.00151572865906509 0.00657389099150725 -0.218432672960972 rpy=0 0 0 -> xyz=0.0015157 0.0059921 -0.21836 rpy=0 0 0
- joint right_shoulder_pitch_joint: limit lower=-0.872665 upper=3.141593 effort=90 velocity=10 -> lower=-0.872665 upper=3.141593 effort=30 velocity=3.98
- joint right_shoulder_roll_joint: limit lower=0 upper=1.570796 effort=75 velocity=10 -> lower=0 upper=1.570796 effort=25 velocity=12.25
- joint right_shoulder_yaw_joint: limit lower=-1.570796 upper=1.570796 effort=60 velocity=10 -> lower=-1.570796 upper=1.570796 effort=20 velocity=5.45
- joint right_wrist_yaw_joint: limit lower=-3.141593 upper=3.141593 effort=36 velocity=10 -> lower=-3.141593 upper=3.141593 effort=12 velocity=9.32
- joint waist_yaw_joint: limit lower=-1.570796 upper=1.570796 effort=120 velocity=10 -> lower=-1.570796 upper=1.570796 effort=40 velocity=12.57
